File: Circuits1/Rx.sch (KiCad schematic (older format))
At the start: 17 parts

Commit message: PCB Layout with 0806
Parts:
- removed X?: QUARTZCMS4, ~, symbol QUARTZCMS4
- added C10: 100nF, ~, symbol C
- added C11: 10uF, ~, symbol C
- added D1: RX, ~, symbol LED
- added D2: LED, ~, symbol LED
- added D3: TX, ~, symbol LED
- added R5, R6, R7: 680, ~, symbol R
- added U2: LD1117, MODULE, symbol LD1117
- added X1: QUARTZ, ~, symbol QUARTZ
- gave numbers to parts that had none: 16
Connections:
- net labels added: 3V3, CE, CSN, MISO, MOSI, SCK
- wire segments 61 -> 89
