File: Circuits1/Tx.kicad_pcb (KiCad board)
At the start: 2 copper layers, 38 x 54 mm, 56 parts, among them CON1 USB-MINI-B, P1 CONN_3X2, SW1 SW_PUSH, SW2 Power Select, U1 ATMEGA32U4, U2 LD1117, U3 NRF24L01+, U4 MPU-6050, X1 QUARTZ, X2 QUARTZ

Commit message: Neatened up for report
Other:
- board size 38 x 54 mm -> 38 x 53.3 mm
Changed lines of the file:
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@@
     (22 B.Mask user)
     (23 F.Mask user)
-    (24 Dwgs.User user)
-    (25 Cmts.User user hide)
+    (24 Dwgs.User user hide)
+    (25 Cmts.User user)
     (26 Eco1.User user)
     (27 Eco2.User user)
@@
     (visible_elements 7FFEFB79)
     (pcbplotparams
-      (layerselection 32769)
+      (layerselection 33587201)
       (usegerberextensions false)
       (excludeedgelayer false)
@@
       (hpglpenoverlay 2)
       (psnegative false)
-      (psa4output true)
+      (psa4output false)
       (plotreference true)
       (plotvalue true)
@@
       (drillshape 1)
       (scaleselection 1)
-      (outputdirectory ""))
+      (outputdirectory ../../Diagrams/))
   )
   (net 0 "")
@@
     (add_net VCC)
   )
+  (module Antenna (layer F.Cu)
+    (at 157.458 70.802 180)
+    (fp_text reference A1 (at 12.99972 -2.49936 180) (layer F.SilkS)
+      (effects (font (size 1.00076 1.00076) (thickness 0.14986)))
+    )
+    (fp_text value Antenna (at 17.00022 7.00024 180) (layer F.SilkS)
+      (effects (font (size 1.00076 1.00076) (thickness 0.14986)))
+    )
+    (fp_line (start -16.80972 -7.22376) (end 12.52982 -7.22376) (layer Dwgs.User) (width 0.6096))
+    (pad "" smd rect (at 2.28092 -3.30454) (size 3.2004 1.20904)
+      (layers F.Cu F.Paste F.Mask)
+    )
+    (pad "" smd rect (at 2.28092 -4.31038) (size 1.19888 0.8001)
+      (layers F.Cu F.Paste F.Mask)
+    )
+    (pad "" smd rect (at -1.9304 -6.31444) (size 25.58034 1.20904)
+      (layers F.Cu F.Paste F.Mask)
+    )
+    (pad "" smd rect (at 6.27126 -5.20954) (size 9.17956 1.00076)
+      (layers F.Cu F.Paste F.Mask)
+    )
+    (pad "" smd rect (at 9.76884 -3.37566) (size 2.17932 2.66954)
+      (layers F.Cu F.Paste F.Mask)
+    )
+    (pad "" smd rect (at 5.77088 -1.39446) (size 10.18032 1.29032)
+      (layers F.Cu F.Paste F.Mask)
+    )
+    (pad 2 smd rect (at 1.28016 -0.381) (size 1.19888 0.73914)
+      (layers F.Cu F.Paste F.Mask)
+      (net 11 GND)
+      (zone_connect 2)
+    )
+    (pad 2 smd rect (at 3.27914 -0.381) (size 1.19888 0.73914)
+      (layers F.Cu F.Paste F.Mask)
+      (net 11 GND)
+      (zone_connect 2)
+    )
+    (pad "" smd rect (at 0.42672 -2.54508 315) (size 0.45974 1.39954)
+      (layers F.Cu F.Paste F.Mask)
+    )
+    (pad 1 smd rect (at 0 -1.10998) (size 0.45974 2.19964)
+      (layers F.Cu F.Paste F.Mask)
+      (net 10 ANTENNA)
+    )
+  )
   (module USB_MINI_B (layer F.Cu)
     (at 178.288 40.309 180)
@@
     )
   )
-  (module Antenna (layer F.Cu)
-    (at 157.458 70.802 180)
-    (fp_text reference A1 (at 12.99972 -2.49936 180) (layer F.SilkS)
-      (effects (font (size 1.00076 1.00076) (thickness 0.14986)))
-    )
-    (fp_text value Antenna (at 17.00022 7.00024 180) (layer F.SilkS)
-      (effects (font (size 1.00076 1.00076) (thickness 0.14986)))
-    )
-    (fp_line (start -16.80972 -7.22376) (end 12.52982 -7.22376) (layer F.SilkS) (width 0.6096))
-    (pad "" smd rect (at 2.28092 -3.30454) (size 3.2004 1.20904)
-      (layers F.Cu F.Paste F.Mask)
-    )
-    (pad "" smd rect (at 2.28092 -4.31038) (size 1.19888 0.8001)
-      (layers F.Cu F.Paste F.Mask)
-    )
-    (pad "" smd rect (at -1.9304 -6.31444) (size 25.58034 1.20904)
-      (layers F.Cu F.Paste F.Mask)
-    )
-    (pad "" smd rect (at 6.27126 -5.20954) (size 9.17956 1.00076)
-      (layers F.Cu F.Paste F.Mask)
-    )
-    (pad "" smd rect (at 9.76884 -3.37566) (size 2.17932 2.66954)
-      (layers F.Cu F.Paste F.Mask)
-    )
-    (pad "" smd rect (at 5.77088 -1.39446) (size 10.18032 1.29032)
-      (layers F.Cu F.Paste F.Mask)
-    )
-    (pad 2 smd rect (at 1.28016 -0.381) (size 1.19888 0.73914)
-      (layers F.Cu F.Paste F.Mask)
-      (net 11 GND)
-      (zone_connect 2)
-    )
-    (pad 2 smd rect (at 3.27914 -0.381) (size 1.19888 0.73914)
-      (layers F.Cu F.Paste F.Mask)
-      (net 11 GND)
-      (zone_connect 2)
-    )
-    (pad "" smd rect (at 0.42672 -2.54508 315) (size 0.45974 1.39954)
-      (layers F.Cu F.Paste F.Mask)
-    )
-    (pad 1 smd rect (at 0 -1.10998) (size 0.45974 2.19964)
-      (layers F.Cu F.Paste F.Mask)
-      (net 10 ANTENNA)
-    )
-  )
   (module Drill3mm   locked (layer F.Cu)
     (at 151.358 51.552)
@@
   )
   (gr_line (start 144.108 78.302) (end 144.108 25.052) (angle 90) (layer Edge.Cuts) (width 0.09906))
-  (gr_line (start 182.088 24.987) (end 144.088 24.987) (angle 90) (layer Edge.Cuts) (width 0.09906))
-  (gr_line (start 182.088 78.987) (end 182.088 24.987) (angle 90) (layer Edge.Cuts) (width 0.09906))
+  (gr_line (start 182.088 25.052) (end 144.108 25.052) (angle 90) (layer Edge.Cuts) (width 0.09906))
+  (gr_line (start 182.088 78.302) (end 182.088 25.052) (angle 90) (layer Edge.Cuts) (width 0.09906))
   (gr_line (start 181.858 51.552) (end 144.108 51.552) (angle 90) (layer Cmts.User) (width 0.20066))
   (gr_line (start 151.358 24.802) (end 151.358 78.302) (angle 90) (layer Cmts.User) (width 0.20066))
@@
     (arrow2b (pts (xy 182.108 88.301999) (xy 180.981497 88.888419)))
   )
-  (gr_line (start 144.108 78.302) (end 182.108 78.302) (angle 90) (layer Edge.Cuts) (width 0.09906))
+  (gr_line (start 144.108 78.302) (end 182.088 78.302) (angle 90) (layer Edge.Cuts) (width 0.09906))
   (segment (start 169.672 49.276) (end 169.672 45.466) (width 0.59944) (layer B.Cu) (net 1))
   (segment (start 169.672 45.466) (end 171.704 43.434) (width 0.59944) (layer B.Cu) (net 1))
@@
   (segment (start 158.75 64.262) (end 158.75 60.96) (width 0.254) (layer F.Cu) (net 9))
   (segment (start 159.766 65.278) (end 158.75 64.262) (width 0.254) (layer F.Cu) (net 9))
-  (via (at 159.766 65.278) (size 1.2) (layers F.Cu B.Cu) (net 9) (status 1000000))
+  (via (at 159.766 65.278) (size 1.2) (layers F.Cu B.Cu) (net 9))
   (segment (start 159.004 60.198) (end 159.004 60.076) (width 0.254) (layer F.Cu) (net 9))
   (segment (start 161.943 61.62816) (end 162.39984 61.62816) (width 0.59944) (layer F.Cu) (net 9))
